Commit message: Adjudicate PC convention: nominal URDF 0/13 violations (origin-inertia checker + bidirectional unit test in dynamics.py); v1.0's 13/13 was a checker bug. Canonical artifact: x1_gmass_anchored.urdf (37.100kg, only base_link mass changed). gm_validate: correct convention, conditional deps, fixed seed (local==remote 37.355kg, dev 0.000kg). Docs: PASS_CRITERIA v1.1 + DELIVERY revised atomically.

File: prime_identify/results/x1_gmass_anchored.urdf (robot description, URDF)
Before this commit: robot x1, 58 links, 57 joints
Links:
- link base_link: mass 6.0811648 -> 6.08146115
- link left_hip_pitch: mass 1.67336544 -> 1.6733645
- link left_hip_roll: mass 0.285621909 -> 0.28562185
- link left_hip_yaw: mass 2.73696232 -> 2.7369623
- link left_knee_pitch: mass 1.68649359 -> 1.5122608
- link right_hip_pitch: mass 1.66657445 -> 1.6665735
- link right_hip_roll: mass 0.287687989 -> 0.28768793
- link right_hip_yaw: mass 2.69635352 -> 2.6963535
- link right_knee_pitch: mass 1.68377278 -> 1.50954
