Commit message: Audit round-4: R9 export artifacts backfilled + stale docstring fixed + sysid_path v1.1 + archived test-run evidence
- spi_identify/export/ regenerated from r9_indomain_params.json via apply_params.py (mass 3.15196154 in URDF/MJCF; DR + report.md updated) — repo export no longer carries stale F1-v15 values; matches T8 remote apply output
- regress.py module docstring: gyro coupling now documented for ALL serial joints with correct magnitudes (knee gyro_rms 0.29 largest serial, hip ~0.19, ankle_roll ~0.009; was stale 'hip joints, knee ~0.007')
- sysid_path.md: route B synced to T10 (all-serial gyro coupling + J2 significance screen); version bumped v1.0 -> v1.1 per its own maintenance rule
- archived local unit-test run evidence: joint_identify/results/unittest_run_2026-09-03.txt (24 tests OK) + spi_identify/results/unittest_run_2026-09-03.txt (68 tests OK) — '24 green' no longer backed only by commit messages
- J1/J2/J3 remain documented next-round boundary (new-data collection required; per steering round-2 instruction 6)

File: spi_identify/export/x1_identified.urdf (robot description, URDF)
Before this commit: robot x1, 58 links, 57 joints
Links:
- link base_link: mass 3.78305736 -> 3.15196154
